File: Elektronik/Drivers/DRV8302Breakout/DRV.sch (KiCad schematic (older format))
At the start: 1 part

Commit message: FirstDriverBegun
Parts:
- removed J?: CONN_02X20, symbol CONN_02X20
- added J?: CONN_CPU, symbol Conn_02x15_Odd_Even
- added J?: Conn_POWER, symbol Conn_02x10_Odd_Even
Connections:
- net labels added: VCC
- wire segments 51 -> 104
Changed lines of the file:
@@
 LIBS:contrib
 LIBS:valves
+LIBS:BLDC_4-cache
+LIBS:BLDC_4-rescue
+LIBS:DRV8302Breakout-cache
 LIBS:DRV-cache
 EELAYER 25 0
@@
 	4450 2650 4800 2650
 Wire Wire Line
-	4450 2750 4800 2750
-Wire Wire Line
-	4800 2850 4450 2850
-Wire Wire Line
-	6650 1350 6200 1350
-Wire Wire Line
-	6650 1450 6200 1450
-Wire Wire Line
-	6650 1550 6200 1550
-Wire Wire Line
-	6650 1650 6200 1650
-Wire Wire Line
-	6200 1750 6650 1750
-Wire Wire Line
-	6650 1850 6200 1850
-Wire Wire Line
-	6650 2000 6200 2000
-Wire Wire Line
-	6650 2100 6200 2100
-Wire Wire Line
-	6650 2200 6200 2200
-Wire Wire Line
-	6650 2400 6200 2400
-Wire Wire Line
-	6650 2500 6200 2500
+	4100 2750 4800 2750
+Wire Wire Line
+	3500 2850 4800 2850
+Wire Wire Line
+	6200 1350 7900 1350
+Wire Wire Line
+	6200 1450 8400 1450
+Wire Wire Line
+	6200 1550 7800 1550
+Wire Wire Line
+	6200 1650 8550 1650
+Wire Wire Line
+	6200 1750 7700 1750
+Wire Wire Line
+	6200 1850 7600 1850
+Wire Wire Line
+	6200 2000 7200 2000
+Wire Wire Line
+	6200 2100 7150 2100
+Wire Wire Line
+	6200 2200 7100 2200
+Wire Wire Line
+	6200 2400 6850 2400
+Wire Wire Line
+	6200 2500 6800 2500
 Wire Wire Line
 	6650 2600 6200 2600
 Wire Wire Line
-	6200 2850 6650 2850
-Wire Wire Line
-	6200 2950 6650 2950
-Wire Wire Line
-	6200 3050 6650 3050
-Wire Wire Line
-	6200 3150 6650 3150
+	6200 2850 7300 2850
+Wire Wire Line
+	6200 2950 7350 2950
+Wire Wire Line
+	6200 3050 7400 3050
+Wire Wire Line
+	6200 3150 7450 3150
 Wire Wire Line
 	2500 1550 2500 2550
@@
 Wire Wire Line
 	2300 3100 2300 3050
+Wire Wire Line
+	2550 1650 2550 3100
+Wire Wire Line
+	2550 3100 2600 3100
+Wire Wire Line
+	2600 3100 2600 3050
+Wire Wire Line
+	2650 1850 2650 3100
+Wire Wire Line
+	2650 3100 2700 3100
+Wire Wire Line
+	2700 3100 2700 3050
+Wire Wire Line
+	2750 2050 2750 3100
+Wire Wire Line
+	2750 3100 2800 3100
+Wire Wire Line
+	2800 3100 2800 3050
+Wire Wire Line
+	2300 2350 2300 2550
+Wire Wire Line
+	2800 1350 2800 2550
+Wire Wire Line
+	2850 2500 2850 3100
+Wire Wire Line
+	2850 3100 2900 3100
+Wire Wire Line
+	2900 3100 2900 3050
 $Comp
-L CONN_02X20 J?
-U 1 1 5AFCE106
-P 2750 2800
-F 0 "J?" H 2750 3850 50  0000 C CNN
-F 1 "CONN_02X20" V 2750 2800 50  0000 C CNN
-F 2 "" H 2750 1850 50  0001 C CNN
-F 3 "" H 2750 1850 50  0001 C CNN
-	1    2750 2800
+L VCC #PWR?
+U 1 1 5AFD4E17
+P 1800 3250
+F 0 "#PWR?" H 1800 3100 50  0001 C CNN
+F 1 "VCC" H 1800 3400 50  0000 C CNN
+F 2 "" H 1800 3250 50  0001 C CNN
+F 3 "" H 1800 3250 50  0001 C CNN
+	1    1800 3250
+	-1   0    0    1
+$EndComp
+Wire Wire Line
+	1800 3250 1800 3050
+Wire Wire Line
+	2100 3050 2050 3050
+Wire Wire Line
+	2050 3050 2050 2400
+Wire Wire Line
+	2050 2400 4450 2400
+Wire Wire Line
+	4450 2400 4450 2650
+Wire Wire Line
+	4100 2750 4100 2450
+Wire Wire Line
+	4100 2450 2100 2450
+Wire Wire Line
+	2100 2450 2100 2550
+$Comp
+L Conn_02x15_Odd_Even J?
+U 1 1 5AFD845E
+P 2500 2850
+F 0 "J?" H 2550 3650 50  0000 C CNN
+F 1 "CONN_CPU" H 2550 2050 50  0000 C CNN
+F 2 "" H 2500 2850 50  0001 C CNN
+F 3 "" H 2500 2850 50  0001 C CNN
+	1    2500 2850
 	0    -1   -1   0
 $EndComp
 Wire Wire Line
-	2550 1650 2550 3100
-Wire Wire Line
-	2550 3100 2600 3100
-Wire Wire Line
-	2600 3100 2600 3050
-Wire Wire Line
-	2650 1850 2650 3100
-Wire Wire Line
-	2650 3100 2700 3100
-Wire Wire Line
-	2700 3100 2700 3050
-Wire Wire Line
-	2750 2050 2750 3100
-Wire Wire Line
-	2750 3100 2800 3100
-Wire Wire Line
-	2800 3100 2800 3050
-Wire Wire Line
-	2300 2350 2300 2550
-Wire Wire Line
-	2800 1350 2800 2550
-Wire Wire Line
-	2850 2500 2850 3100
-Wire Wire Line
-	2850 3100 2900 3100
-Wire Wire Line
-	2900 3100 2900 3050
+	3500 2850 3500 3200
+Wire Wire Line
+	3500 3200 2400 3200
+Wire Wire Line
+	2400 3200 2400 3050
+$Comp
+L Conn_02x10_Odd_Even J?
+U 1 1 5AFDA65D
+P 8100 2250
+F 0 "J?" H 8150 2750 50  0000 C CNN
+F 1 "Conn_POWER" H 8150 1650 50  0000 C CNN
+F 2 "" H 8100 2250 50  0001 C CNN
+F 3 "" H 8100 2250 50  0001 C CNN
+	1    8100 2250
+	1    0    0    -1
+$EndComp
+Wire Wire Line
+	7900 1350 7900 1850
+Wire Wire Line
+	8400 1450 8400 1850
+Wire Wire Line
+	7900 1950 7800 1950
+Wire Wire Line
+	7800 1950 7800 1550
+Wire Wire Line
+	8550 1650 8550 1950
+Wire Wire Line
+	8550 1950 8400 1950
+Wire Wire Line
+	7700 1750 7700 2050
+Wire Wire Line
+	7700 2050 7900 2050
+Wire Wire Line
+	7600 1850 7600 1700
+Wire Wire Line
+	7600 1700 8650 1700
+Wire Wire Line
+	8650 1700 8650 2050
+Wire Wire Line
+	8650 2050 8400 2050
+Wire Wire Line
+	7900 2350 7300 2350
+Wire Wire Line
+	7300 2350 7300 2850
+Wire Wire Line
+	7350 2950 7350 2400
+Wire Wire Line
+	7350 2400 8500 2400
+Wire Wire Line
+	8500 2400 8500 2350
+Wire Wire Line
+	8500 2350 8400 2350
+Wire Wire Line
+	7400 3050 7400 2450
+Wire Wire Line
+	7400 2450 7900 2450
+Wire Wire Line
+	7450 3150 7450 2500
+Wire Wire Line
+	7450 2500 8500 2500
+Wire Wire Line
+	8500 2500 8500 2450
+Wire Wire Line
+	8500 2450 8400 2450
+Wire Wire Line
+	7900 2550 7200 2550
+Wire Wire Line
+	7200 2550 7200 2000
+Wire Wire Line
+	7900 2650 7150 2650
+Wire Wire Line
+	7150 2650 7150 2100
+Wire Wire Line
+	7100 2200 7100 2750
+Wire Wire Line
+	7100 2750 7900 2750
+Wire Wire Line
+	8400 2550 8450 2550
+Wire Wire Line
+	8450 2550 8450 2600
+Wire Wire Line
+	8450 2600 6850 2600
+Wire Wire Line
+	6850 2600 6850 2400
+Wire Wire Line
+	6800 2500 6800 2700
+Wire Wire Line
+	6800 2700 8450 2700
+Wire Wire Line
+	8450 2700 8450 2650
+Wire Wire Line
+	8450 2650 8400 2650
+Wire Wire Line
+	8400 2750 8500 2750
+Wire Wire Line
+	8500 2750 8500 2800
+Wire Wire Line
+	8500 2800 6650 2800
+Wire Wire Line
+	6650 2800 6650 2600
 $EndSCHEMATC

Commit message: fewChanges
Changed lines of the file:
@@
 $Descr A4 11693 8268
 encoding utf-8
-Sheet 1 2
+Sheet 1 3
 Title ""
 Date ""
@@
 Wire Wire Line
 	6650 2800 6650 2600
+$Sheet
+S 4800 3500 600  300
+U 5AFDF8CF
+F0 "Voltreg" 60
+F1 "VoltageReg.sch" 60
+F2 "VIN" I R 5400 3650 60
+F3 "12V" I L 4800 3650 60
+$EndSheet
+Wire Wire Line
+	4750 3650 1900 3650
+Wire Wire Line
+	1900 3650 1900 3050
+Text GLabel 5950 3650 2    60   Input ~ 0
+V_SUPPLY
+Wire Wire Line
+	5400 3650 5950 3650
 $EndSCHEMATC
