File: Elektronik/Drivers/Power/suppliesFrom60V.sch (KiCad schematic (older format))
At the start: 11 parts

Commit message: fewChanges
Connections:
- net +VDC: now reaches C1.1, Ureg?.7 (VIN)
Changed lines of the file:
@@
 LIBS:contrib
 LIBS:valves
+LIBS:suppliesFrom60V-cache
 EELAYER 25 0
 EELAYER END
@@
 Wire Wire Line
 	5050 4500 4350 4500
+$Comp
+L +VDC #PWR?
+U 1 1 5AFE02E8
+P 6850 3700
+F 0 "#PWR?" H 6850 3600 50  0001 C CNN
+F 1 "+VDC" H 6850 3950 50  0000 C CNN
+F 2 "" H 6850 3700 50  0001 C CNN
+F 3 "" H 6850 3700 50  0001 C CNN
+	1    6850 3700
+	1    0    0    -1
+$EndComp
+Wire Wire Line
+	6850 3850 6850 3700
 $EndSCHEMATC
