File: Elektronik/CPUs/CJMCU_STM32F407_Breakout.sch (KiCad schematic (older format))
At the start: 5 parts

Commit message: firstStm42f4
Parts:
- added J?: CONN_HALL, symbol CONN_01X05
- added J?: CONN_Incremental, symbol CONN_01X05
- added J?: Connector_StepDirI²CSPIUART, symbol CONN_01X06
- added J?: Analog_In, symbol CONN_01X02
- J?: value Hall_conn -> Encoder
Connections:
- wire segments 73 -> 74
Changed lines of the file:
@@
 P 8450 4350
 F 0 "J?" H 8450 4650 50  0000 C CNN
-F 1 "Hall_conn" V 8550 4350 50  0000 C CNN
+F 1 "Encoder" V 8550 4350 50  0000 C CNN
 F 2 "" H 8450 4350 50  0001 C CNN
 F 3 "" H 8450 4350 50  0001 C CNN
@@
 Wire Wire Line
 	7100 4100 7100 5450
+$Comp
+L CONN_01X05 J?
+U 1 1 5B0D0A44
+P 4750 4450
+F 0 "J?" H 4750 4750 50  0000 C CNN
+F 1 "CONN_HALL" V 4850 4450 50  0000 C CNN
+F 2 "" H 4750 4450 50  0001 C CNN
+F 3 "" H 4750 4450 50  0001 C CNN
+	1    4750 4450
+	1    0    0    -1
+$EndComp
+$Comp
+L CONN_01X05 J?
+U 1 1 5B0D0E20
+P 4750 3750
+F 0 "J?" H 4750 4050 50  0000 C CNN
+F 1 "CONN_Incremental" V 4850 3750 50  0000 C CNN
+F 2 "" H 4750 3750 50  0001 C CNN
+F 3 "" H 4750 3750 50  0001 C CNN
+	1    4750 3750
+	1    0    0    1
+$EndComp
+$Comp
+L CONN_01X06 J?
+U 1 1 5B0D0E7E
+P 6500 2250
+F 0 "J?" H 6500 2600 50  0000 C CNN
+F 1 "Connector_StepDirI²CSPIUART" V 6600 2250 50  0000 C CNN
+F 2 "" H 6500 2250 50  0001 C CNN
+F 3 "" H 6500 2250 50  0001 C CNN
+	1    6500 2250
+	0    -1   -1   0
+$EndComp
+$Comp
+L CONN_01X02 J?
+U 1 1 5B0D1189
+P 7600 2350
+F 0 "J?" H 7600 2500 50  0000 C CNN
+F 1 "Analog_In" V 7700 2350 50  0000 C CNN
+F 2 "" H 7600 2350 50  0001 C CNN
+F 3 "" H 7600 2350 50  0001 C CNN
+	1    7600 2350
+	0    -1   -1   0
+$EndComp
+$Comp
+L GND #PWR?
+U 1 1 5B0D1378
+P 7650 2600
+F 0 "#PWR?" H 7650 2350 50  0001 C CNN
+F 1 "GND" H 7650 2450 50  0000 C CNN
+F 2 "" H 7650 2600 50  0001 C CNN
+F 3 "" H 7650 2600 50  0001 C CNN
+	1    7650 2600
+	1    0    0    -1
+$EndComp
+Wire Wire Line
+	7650 2550 7650 2600
 $EndSCHEMATC
